File: Croketa.kicad_pcb (KiCad board)
At the start: 2 copper layers, 17.8 x 33 mm, 5 parts, among them P1 Digital, P2 COM, P3 ADC, P4 Analog, P5 ADC

Commit message: first components places
Parts:
- removed P2: COM, Socket_Arduino_Pro_Mini:Socket_Strip_Arduino_1x06
- removed P5: ADC, Socket_Arduino_Pro_Mini:Socket_Strip_Arduino_1x02
- added C1: 1uF, Capacitor_SMD:C_0805_2012Metric_Pad1.15x1.40mm_HandSolder, F.Cu at (184.3, 87.6)
- added C2: 2.2uF, Capacitor_SMD:C_0805_2012Metric_Pad1.15x1.40mm_HandSolder, F.Cu at (180.6, 87.6)
- added C3: 0.1uF, Capacitor_SMD:C_0805_2012Metric_Pad1.15x1.40mm_HandSolder, F.Cu at (174.3, 94.6)
- added C4: 0.1uF, Capacitor_SMD:C_0805_2012Metric_Pad1.15x1.40mm_HandSolder, F.Cu at (178.1, 90.5)
- added C5: 0.1uF, Capacitor_SMD:C_0805_2012Metric_Pad1.15x1.40mm_HandSolder, F.Cu at (178.1, 92.4)
- added D1: LED, LED_SMD:LED_0805_2012Metric_Pad1.15x1.40mm_HandSolder, F.Cu at (180.6, 85.7)
- added D2: LED, LED_SMD:LED_0805_2012Metric_Pad1.15x1.40mm_HandSolder, F.Cu at (185.5, 82.3)
- added D3: LED, LED_SMD:LED_0805_2012Metric_Pad1.15x1.40mm_HandSolder, F.Cu at (174.3, 92.6)
- added D4: LED, LED_SMD:LED_0805_2012Metric_Pad1.15x1.40mm_HandSolder, F.Cu at (174.3, 90.5)
- added F1: 500mA, Fuse:Fuse_0805_2012Metric_Pad1.15x1.40mm_HandSolder, F.Cu at (184.4, 85.6)
- added J1: USB_B_Micro, Connector_USB:USB_Micro-B_Wuerth_629105150521, F.Cu at (173.7, 84.6)
- added J2: CORTEX_DEBUGPTH, Connector_PinHeader_2.54mm:PinHeader_2x05_P2.54mm_Vertical, F.Cu at (164.4, 83.1)
- added JP1: Jumper_NC_Small, Connector_PinHeader_2.54mm:PinHeader_1x02_P2.54mm_Vertical, F.Cu at (170.6, 91.3)
- added R1: 330, Resistor_SMD:R_0805_2012Metric_Pad1.15x1.40mm_HandSolder, F.Cu at (178.1, 94.4)
- added R2: 330, Resistor_SMD:R_0805_2012Metric_Pad1.15x1.40mm_HandSolder, F.Cu at (181.8, 89.6)
- added R3: 330, Resistor_SMD:R_0805_2012Metric_Pad1.15x1.40mm_HandSolder, F.Cu at (181.8, 91.5)
- added R4: 330, Resistor_SMD:R_0805_2012Metric_Pad1.15x1.40mm_HandSolder, F.Cu at (181.8, 93.5)
- added SW1: SW_DPST_x2, Button_Switch_SMD:SW_SPST_B3U-1000P-B, F.Cu at (181.1, 83.0)
- added U1: AP2112K-3.3TRG1, Package_TO_SOT_SMD:SOT-23-5, F.Cu at (187.4, 108.5)
- added U2: ATSAMD21E18A-AF, Package_QFP:LQFP-32_7x7mm_P0.8mm, F.Cu at (180.4, 111.8)
- P3: value ADC -> Analog
- moved P3 11.7 mm to (142.2, 86.4)
Connections:
- P3 pad 1: /A5 -> /RAW
- P3 pad 2: /A4 -> GND
