File: Croketa.sch (KiCad schematic (older format))
At the start: 25 parts, among them P1 Digital, P2 COM, P3 ADC, P4 Analog, P5 ADC

Commit message: Schematic finished
Parts:
- removed P2: COM, Socket_Arduino_Pro_Mini:Socket_Strip_Arduino_1x06, symbol Connector_Generic:Conn_01x06
- removed P5: ADC, Socket_Arduino_Pro_Mini:Socket_Strip_Arduino_1x02, symbol Connector_Generic:Conn_01x02
- added J?: CORTEX_DEBUGPTH, symbol Connector_Generic:Conn_02x05_Odd_Even
- added SW?: SW_DPST_x2, symbol Switch:SW_DPST_x2
Connections:
- net labels removed: A5, A6, A7, DTR
- wire segments 114 -> 120
- no-connect marks 0 -> 4

Commit message: Schematic finished, now yes
Parts:
- removed L?: 30Ohm, symbol Device:L
- removed R?: 10K, symbol Device:R
- F1: renamed from F?; value Polyfuse -> 500mA
- gave numbers to parts that had none: 19
- renumbered P3 to P2, P4 to P3
Connections:
- wire segments 120 -> 114

Commit message: first components places
Parts:
- removed J2: CORTEX_DEBUGPTH, symbol Connector_Generic:Conn_02x05_Odd_Even
- added J2: Conn_01x04, Connector_PinHeader_2.54mm:PinHeader_1x04_P2.54mm_Vertical, symbol Connector_Generic:Conn_01x04
- C1, C2, C3, C4, C5: footprint (none) -> Capacitor_SMD:C_0805_2012Metric_Pad1.15x1.40mm_HandSolder
- D1, D2, D3, D4: footprint (none) -> LED_SMD:LED_0805_2012Metric_Pad1.15x1.40mm_HandSolder
- F1: footprint (none) -> Fuse:Fuse_0805_2012Metric_Pad1.15x1.40mm_HandSolder
- J1: footprint (none) -> Connector_USB:USB_Micro-B_Wuerth_629105150521
- JP1: footprint (none) -> Connector_PinHeader_2.54mm:PinHeader_1x02_P2.54mm_Vertical
- P1: footprint Socket_Arduino_Pro_Mini:Socket_Strip_Arduino_1x12 -> Connector_PinHeader_2.54mm:PinHeader_1x12_P2.54mm_Vertical
- R1: renamed from R2; footprint (none) -> Resistor_SMD:R_0805_2012Metric_Pad1.15x1.40mm_HandSolder
- R2: renamed from R3; footprint (none) -> Resistor_SMD:R_0805_2012Metric_Pad1.15x1.40mm_HandSolder
- R3: renamed from R4; footprint (none) -> Resistor_SMD:R_0805_2012Metric_Pad1.15x1.40mm_HandSolder
- R4: renamed from R5; footprint (none) -> Resistor_SMD:R_0805_2012Metric_Pad1.15x1.40mm_HandSolder
- SW1: footprint (none) -> Button_Switch_SMD:SW_SPST_B3U-1000P-B
- U1: footprint SOT95P285X140-5N -> Package_TO_SOT_SMD:SOT-23-5
- U2: footprint QFP80P900X900X120-32N -> Package_QFP:LQFP-32_7x7mm_P0.8mm
Connections:
- wire segments 114 -> 108
- no-connect marks 4 -> 0

Commit message: Second arrangement of components in pcb
Parts:
- removed J2: Conn_01x04, Connector_PinHeader_2.54mm:PinHeader_1x04_P2.54mm_Vertical, symbol Connector_Generic:Conn_01x04
- added J2: Conn_02x02_Odd_Even, Connector_PinHeader_2.54mm:PinHeader_2x02_P2.54mm_Vertical_SMD, symbol Connector_Generic:Conn_02x02_Odd_Even
Changed lines of the file:
@@
 L power:+3.3V #PWR016
 U 1 1 5BB866B1
-P 9850 3250
-F 0 "#PWR016" H 9850 3100 50  0001 C CNN
-F 1 "+3.3V" H 9865 3423 50  0000 C CNN
-F 2 "" H 9850 3250 50  0001 C CNN
-F 3 "" H 9850 3250 50  0001 C CNN
-	1    9850 3250
+P 9600 3880
+F 0 "#PWR016" H 9600 3730 50  0001 C CNN
+F 1 "+3.3V" H 9615 4053 50  0000 C CNN
+F 2 "" H 9600 3880 50  0001 C CNN
+F 3 "" H 9600 3880 50  0001 C CNN
+	1    9600 3880
 	1    0    0    -1
 $EndComp
@@
 L power:GND #PWR015
 U 1 1 5BB89DC5
-P 9640 3420
-F 0 "#PWR015" H 9640 3170 50  0001 C CNN
-F 1 "GND" H 9640 3270 50  0000 C CNN
-F 2 "" H 9640 3420 50  0000 C CNN
-F 3 "" H 9640 3420 50  0000 C CNN
-	1    9640 3420
+P 10700 3910
+F 0 "#PWR015" H 10700 3660 50  0001 C CNN
+F 1 "GND" H 10700 3760 50  0000 C CNN
+F 2 "" H 10700 3910 50  0000 C CNN
+F 3 "" H 10700 3910 50  0000 C CNN
+	1    10700 3910
 	1    0    0    -1
 $EndComp
-Text Label 9950 3520 2    50   ~ 0
+Text Label 9830 4010 2    50   ~ 0
 SWDIO
-Text Label 9950 3620 2    50   ~ 0
+Text Label 10330 4010 0    50   ~ 0
 SWCLK
 Wire Wire Line
@@
 	3950 1410 4430 1410
 $Comp
-L Connector_Generic:Conn_01x04 J2
-U 1 1 5BB41D79
-P 10150 3420
-F 0 "J2" H 10230 3412 50  0000 L CNN
-F 1 "Conn_01x04" H 10230 3321 50  0000 L CNN
-F 2 "Connector_PinHeader_2.54mm:PinHeader_1x04_P2.54mm_Vertical" H 10150 3420 50  0001 C CNN
-F 3 "~" H 10150 3420 50  0001 C CNN
-	1    10150 3420
+L Connector_Generic:Conn_02x02_Odd_Even J2
+U 1 1 5BB5EF14
+P 10030 3910
+F 0 "J2" H 10080 4127 50  0000 C CNN
+F 1 "Conn_02x02_Odd_Even" H 10080 4036 50  0000 C CNN
+F 2 "Connector_PinHeader_2.54mm:PinHeader_2x02_P2.54mm_Vertical_SMD" H 10030 3910 50  0001 C CNN
+F 3 "~" H 10030 3910 50  0001 C CNN
+	1    10030 3910
 	1    0    0    -1
 $EndComp
 Wire Wire Line
-	9850 3250 9850 3320
+	9830 3910 9600 3910
 Wire Wire Line
-	9850 3320 9950 3320
+	9600 3910 9600 3880
 Wire Wire Line
-	9640 3420 9950 3420
+	10330 3910 10700 3910
 $EndSCHEMATC

Commit message: Remove leds and change pins I2C
Parts:
- removed D3, D4: LED, LED_SMD:LED_0805_2012Metric_Pad1.15x1.40mm_HandSolder, symbol Device:LED
- removed JP1: Jumper_NC_Small, Connector_PinHeader_2.54mm:PinHeader_1x02_P2.54mm_Vertical, symbol Device:Jumper_NC_Small
- removed R3, R4: 330, Resistor_SMD:R_0805_2012Metric_Pad1.15x1.40mm_HandSolder, symbol Device:R
- D1: value LED -> POWER
Connections:
- net labels added: LED
- net labels removed: RX_LED, TX_LED, USB_HOST_EN
- wire segments 108 -> 101
- no-connect marks 0 -> 1
Other:
- note added: "SAMD21"
- note added: "SOURCE"
- note added: "USB & SWD PORT"

Commit message: V0.2 Fix Connection
Connections:
- net labels added: D+, D-
- net labels removed: +5V, A4, AREF, Reset, USB_D+, USB_D-
- wire segments 101 -> 107
Changed lines of the file:
@@
 Sheet 1 1
 Title "Bast Pro Mini M0"
-Date "2018-09-28"
-Rev "0.1"
+Date "2018-10-08"
+Rev "0.2"
 Comp "Electronic Cats"
 Comment1 "Edgar Capuchino"
-Comment2 ""
+Comment2 "Andrés Sabas"
 Comment3 ""
 Comment4 ""
 $EndDescr
-Text Label 2530 1170 1    60   ~ 0
-RAW
 Text Label 1180 1270 0    60   ~ 0
 1(Tx)
@@
 0(Rx)
 Text Label 1180 1470 0    60   ~ 0
-Reset
+RESET
 Text Label 2680 1470 0    60   ~ 0
-Reset
+RESET
 Text Label 1180 1670 0    60   ~ 0
 2
@@
 	1530 2370 1180 2370
 Wire Wire Line
-	2530 1170 2530 1270
+	2530 1170 2530 1220
 Wire Wire Line
 	2530 1270 2430 1270
@@
 L power:VCC #PWR05
 U 1 1 56D75A9D
-P 2630 1170
-F 0 "#PWR05" H 2630 1020 50  0001 C CNN
-F 1 "VCC" H 2630 1320 50  0000 C CNN
-F 2 "" H 2630 1170 50  0000 C CNN
-F 3 "" H 2630 1170 50  0000 C CNN
-	1    2630 1170
+P 2370 1145
+F 0 "#PWR05" H 2370 995 50  0001 C CNN
+F 1 "VCC" H 2370 1295 50  0000 C CNN
+F 2 "" H 2370 1145 50  0000 C CNN
+F 3 "" H 2370 1145 50  0000 C CNN
+	1    2370 1145
 	1    0    0    -1
 $EndComp
@@
 Wire Wire Line
 	4300 1810 4430 1810
-Text Label 4290 1910 2    50   ~ 0
-AREF
 Wire Wire Line
 	4290 1910 4430 1910
@@
 Wire Wire Line
 	4230 2610 4430 2610
-Text Label 4230 2710 2    60   ~ 0
-A4
 Wire Wire Line
 	4230 2710 4430 2710
@@
 SCL
 Text Label 5890 2310 0    50   ~ 0
-USB_D-
+D-
 Wire Wire Line
 	5630 2310 5890 2310
 Text Label 5910 2410 0    50   ~ 0
-USB_D+
+D+
 Wire Wire Line
 	5630 2410 5910 2410
 Wire Wire Line
 	5630 2510 5890 2510
-Text Label 5890 2510 0    50   ~ 0
-LED
 Wire Wire Line
 	5630 2710 5880 2710
@@
 Wire Wire Line
 	2260 4200 2260 4070
-$Comp
-L power:+5V #PWR03
-U 1 1 5BB50E86
-P 2260 4070
-F 0 "#PWR03" H 2260 3920 50  0001 C CNN
-F 1 "+5V" H 2275 4243 50  0000 C CNN
-F 2 "" H 2260 4070 50  0001 C CNN
-F 3 "" H 2260 4070 50  0001 C CNN
-	1    2260 4070
-	1    0    0    -1
-$EndComp
-$Comp
-L power:+5V #PWR06
-U 1 1 5BB50EF0
-P 7900 4380
-F 0 "#PWR06" H 7900 4230 50  0001 C CNN
-F 1 "+5V" H 7915 4553 50  0000 C CNN
-F 2 "" H 7900 4380 50  0001 C CNN
-F 3 "" H 7900 4380 50  0001 C CNN
-	1    7900 4380
-	1    0    0    -1
-$EndComp
 $Comp
 L Device:C_Small C1
@@
 $EndComp
 Text Label 9945 1730 2    60   ~ 0
-Reset
+RESET
 $Comp
 L power:GND #PWR08
@@
 Text Label 2680 2170 0    50   ~ 0
 12(MISO)
-NoConn ~ 5630 2610
 Wire Notes Line
 	11210 3615 11210 3595
@@
 Text Notes 2665 3775 0    50   ~ 0
 USB & SWD PORT
+Wire Wire Line
+	1550 4400 1730 4400
+Wire Wire Line
+	1550 4500 1730 4500
+NoConn ~ 1550 4600
+Text Label 1730 4400 0    50   ~ 0
+D+
+Text Label 1730 4500 0    50   ~ 0
+D-
+Wire Wire Line
+	5630 2610 5880 2610
+Text Label 5880 2610 0    50   ~ 0
+7
+Text Label 5890 2510 0    50   ~ 0
+6(**)
+Text Label 4230 2710 0    50   ~ 0
+LED
+$Comp
+L Croketa-cache:+3.3V #PWR0101
+U 1 1 5BBD0E40
+P 2630 1170
+F 0 "#PWR0101" H 2630 1020 50  0001 C CNN
+F 1 "+3.3V" H 2645 1343 50  0000 C CNN
+F 2 "" H 2630 1170 50  0001 C CNN
+F 3 "" H 2630 1170 50  0001 C CNN
+	1    2630 1170
+	1    0    0    -1
+$EndComp
+$Comp
+L power:VCC #PWR0102
+U 1 1 5BBD1305
+P 2260 4070
+F 0 "#PWR0102" H 2260 3920 50  0001 C CNN
+F 1 "VCC" H 2277 4243 50  0000 C CNN
+F 2 "" H 2260 4070 50  0001 C CNN
+F 3 "" H 2260 4070 50  0001 C CNN
+	1    2260 4070
+	1    0    0    -1
+$EndComp
+$Comp
+L power:VCC #PWR0103
+U 1 1 5BBD1622
+P 7900 4380
+F 0 "#PWR0103" H 7900 4230 50  0001 C CNN
+F 1 "VCC" H 7917 4553 50  0000 C CNN
+F 2 "" H 7900 4380 50  0001 C CNN
+F 3 "" H 7900 4380 50  0001 C CNN
+	1    7900 4380
+	1    0    0    -1
+$EndComp
+Text Label 2530 1170 1    50   ~ 0
+RAW
+Wire Wire Line
+	2370 1145 2370 1220
+Wire Wire Line
+	2370 1220 2530 1220
+Connection ~ 2530 1220
+Wire Wire Line
+	2530 1220 2530 1270
 $EndSCHEMATC
