File: Croketa.sch (KiCad schematic (older format))
At the start: 18 parts, among them J1 USB_B_Micro, J2 Conn_02x02_Odd_Even, P1 Digital, P2 ADC, P3 Analog, SW1 SW_DPST_x2, U1 AP2112K-3.3TRG1, U2 ATSAMD21E18A-AF

Commit message: New pcb's Bast
Parts:
- C1, C2, C3, C4, C5: footprint Capacitor_SMD:C_0805_2012Metric_Pad1.15x1.40mm_HandSolder -> Capacitor_SMD:C_0603_1608Metric_Pad1.05x0.95mm_HandSolder
- R1, R2: footprint Resistor_SMD:R_0805_2012Metric_Pad1.15x1.40mm_HandSolder -> Resistor_SMD:R_0603_1608Metric_Pad1.05x0.95mm_HandSolder
Changed lines of the file:
@@
 F 0 "C5" H 7272 1166 50  0000 L CNN
 F 1 "0.1uF" H 7272 1075 50  0000 L CNN
-F 2 "Capacitor_SMD:C_0805_2012Metric_Pad1.15x1.40mm_HandSolder" H 7180 1120 50  0001 C CNN
+F 2 "Capacitor_SMD:C_0603_1608Metric_Pad1.05x0.95mm_HandSolder" H 7180 1120 50  0001 C CNN
 F 3 "~" H 7180 1120 50  0001 C CNN
 	1    7180 1120
@@
 F 0 "C4" H 7032 1286 50  0000 L CNN
 F 1 "0.1uF" H 7032 1195 50  0000 L CNN
-F 2 "Capacitor_SMD:C_0805_2012Metric_Pad1.15x1.40mm_HandSolder" H 6940 1240 50  0001 C CNN
+F 2 "Capacitor_SMD:C_0603_1608Metric_Pad1.05x0.95mm_HandSolder" H 6940 1240 50  0001 C CNN
 F 3 "~" H 6940 1240 50  0001 C CNN
 	1    6940 1240
@@
 F 0 "C3" H 6772 1806 50  0000 L CNN
 F 1 "0.1uF" H 6772 1715 50  0000 L CNN
-F 2 "Capacitor_SMD:C_0805_2012Metric_Pad1.15x1.40mm_HandSolder" H 6680 1760 50  0001 C CNN
+F 2 "Capacitor_SMD:C_0603_1608Metric_Pad1.05x0.95mm_HandSolder" H 6680 1760 50  0001 C CNN
 F 3 "~" H 6680 1760 50  0001 C CNN
 	1    6680 1760
@@
 F 0 "R1" H 8630 2121 50  0000 L CNN
 F 1 "330" H 8630 2030 50  0000 L CNN
-F 2 "Resistor_SMD:R_0805_2012Metric_Pad1.15x1.40mm_HandSolder" V 8490 2075 50  0001 C CNN
+F 2 "Resistor_SMD:R_0603_1608Metric_Pad1.05x0.95mm_HandSolder" V 8490 2075 50  0001 C CNN
 F 3 "~" H 8560 2075 50  0001 C CNN
 	1    8560 2075
@@
 F 0 "R2" H 9250 2131 50  0000 L CNN
 F 1 "330" H 9250 2040 50  0000 L CNN
-F 2 "Resistor_SMD:R_0805_2012Metric_Pad1.15x1.40mm_HandSolder" V 9110 2085 50  0001 C CNN
+F 2 "Resistor_SMD:R_0603_1608Metric_Pad1.05x0.95mm_HandSolder" V 9110 2085 50  0001 C CNN
 F 3 "~" H 9180 2085 50  0001 C CNN
 	1    9180 2085
@@
 F 0 "C1" H 8102 4896 50  0000 L CNN
 F 1 "1uF" H 8102 4805 50  0000 L CNN
-F 2 "Capacitor_SMD:C_0805_2012Metric_Pad1.15x1.40mm_HandSolder" H 8010 4850 50  0001 C CNN
+F 2 "Capacitor_SMD:C_0603_1608Metric_Pad1.05x0.95mm_HandSolder" H 8010 4850 50  0001 C CNN
 F 3 "~" H 8010 4850 50  0001 C CNN
 	1    8010 4850
@@
 F 0 "C2" H 10242 4716 50  0000 L CNN
 F 1 "2.2uF" H 10242 4625 50  0000 L CNN
-F 2 "Capacitor_SMD:C_0805_2012Metric_Pad1.15x1.40mm_HandSolder" H 10150 4670 50  0001 C CNN
+F 2 "Capacitor_SMD:C_0603_1608Metric_Pad1.05x0.95mm_HandSolder" H 10150 4670 50  0001 C CNN
 F 3 "~" H 10150 4670 50  0001 C CNN
 	1    10150 4670
