File: Hw/Bast-Pro-Mini-M0.sch (KiCad schematic (older format))
At the start: 18 parts, among them J1 USB_B_Micro, J2 Conn_02x02_Odd_Even, P1 Digital, P2 ADC, P3 Analog, SW1 SW_DPST_x2, U1 AP2112K-3.3TRG1, U2 ATSAMD21E18A-AF

Commit message: Change type of button
Parts:
- SW1: footprint Button_Switch_SMD:SW_SPST_B3U-1000P-B -> Button_Switch_SMD:SW_SPST_TL3342
Changed lines of the file:
@@
 F 0 "SW1" H 10145 1965 50  0000 C CNN
 F 1 "SW_DPST_x2" H 10145 1874 50  0000 C CNN
-F 2 "Button_Switch_SMD:SW_SPST_B3U-1000P-B" H 10145 1730 50  0001 C CNN
+F 2 "Button_Switch_SMD:SW_SPST_TL3342" H 10145 1730 50  0001 C CNN
 F 3 "" H 10145 1730 50  0001 C CNN
 F 4 "B3U-1000P-B" H 10145 1730 50  0001 C CNN "manf#"

Commit message: Updates
Parts:
- C1, C2, C3, C4, C5: symbol Device:C_Small -> Bast-Pro-Mini-M0-rescue:C_Small-Device
- D1, D2: symbol Device:LED -> Bast-Pro-Mini-M0-rescue:LED-Device
- F1: symbol Device:Polyfuse -> Bast-Pro-Mini-M0-rescue:Polyfuse-Device
- J1: symbol Connector:USB_B_Micro -> Bast-Pro-Mini-M0-rescue:USB_B_Micro-Connector
- J2: symbol Connector_Generic:Conn_02x02_Odd_Even -> Bast-Pro-Mini-M0-rescue:Conn_02x02_Odd_Even-Connector_Generic
- P1, P3: symbol Connector_Generic:Conn_01x12 -> Bast-Pro-Mini-M0-rescue:Conn_01x12-Connector_Generic
- P2: symbol Connector_Generic:Conn_01x02 -> Bast-Pro-Mini-M0-rescue:Conn_01x02-Connector_Generic
- R1, R2: symbol Device:R -> Bast-Pro-Mini-M0-rescue:R-Device
- SW1: symbol Switch:SW_DPST_x2 -> Bast-Pro-Mini-M0-rescue:SW_DPST_x2-Switch
- U1: symbol Bast-Pro-Mini-M0-rescue:AP2112K-3.3TRG1-Croketa-cache -> Bast-Pro-Mini-M0-rescue:AP2112K-3.3TRG1-Croketa-cache-Bast-Pro-Mini-M0-rescue
- U2: symbol Bast-Pro-Mini-M0-rescue:ATSAMD21E18A-AF-Croketa-cache -> Bast-Pro-Mini-M0-rescue:ATSAMD21E18A-AF-Croketa-cache-Bast-Pro-Mini-M0-rescue
Changed lines of the file:
@@
-EESchema Schematic File Version 4
+EESchema Schematic File Version 5
 LIBS:Bast-Pro-Mini-M0-cache
-EELAYER 26 0
+EELAYER 29 0
 EELAYER END
 $Descr A4 11693 8268
@@
 	9700 650  9700 475
 $Comp
-L Connector_Generic:Conn_01x02 P2
+L Bast-Pro-Mini-M0-rescue:Conn_01x02-Connector_Generic P2
 U 1 1 56D74FB3
 P 1970 2760
@@
 $EndComp
 $Comp
-L Connector_Generic:Conn_01x12 P1
+L Bast-Pro-Mini-M0-rescue:Conn_01x12-Connector_Generic P1
 U 1 1 56D754D1
 P 1730 1770
@@
 $EndComp
 $Comp
-L Connector_Generic:Conn_01x12 P3
+L Bast-Pro-Mini-M0-rescue:Conn_01x12-Connector_Generic P3
 U 1 1 56D755F3
 P 2230 1770
@@
 1
 $Comp
-L Bast-Pro-Mini-M0-rescue:ATSAMD21E18A-AF-Croketa-cache U2
+L Bast-Pro-Mini-M0-rescue:ATSAMD21E18A-AF-Croketa-cache-Bast-Pro-Mini-M0-rescue U2
 U 1 1 5BAEC202
 P 5030 2010
@@
 	5630 2810 5880 2810
 $Comp
-L Device:C_Small C5
+L Bast-Pro-Mini-M0-rescue:C_Small-Device C5
 U 1 1 5BB06F9B
 P 7180 1120
@@
 $EndComp
 $Comp
-L Device:C_Small C4
+L Bast-Pro-Mini-M0-rescue:C_Small-Device C4
 U 1 1 5BB0701E
 P 6940 1240
@@
 	6940 1110 5630 1110
 $Comp
-L Device:C_Small C3
+L Bast-Pro-Mini-M0-rescue:C_Small-Device C3
 U 1 1 5BB0CC95
 P 6680 1760
@@
 RESET
 $Comp
-L Device:LED D1
+L Bast-Pro-Mini-M0-rescue:LED-Device D1
 U 1 1 5BB1D4DB
 P 8560 1655
@@
 $EndComp
 $Comp
-L Device:LED D2
+L Bast-Pro-Mini-M0-rescue:LED-Device D2
 U 1 1 5BB1D525
 P 9180 1655
@@
 $EndComp
 $Comp
-L Device:R R1
+L Bast-Pro-Mini-M0-rescue:R-Device R1
 U 1 1 5BB1D679
 P 8560 2075
@@
 $EndComp
 $Comp
-L Device:R R2
+L Bast-Pro-Mini-M0-rescue:R-Device R2
 U 1 1 5BB1D85A
 P 9180 2085
@@
 LED
 $Comp
-L Connector:USB_B_Micro J1
+L Bast-Pro-Mini-M0-rescue:USB_B_Micro-Connector J1
 U 1 1 5BB47277
 P 1250 4400
@@
 Connection ~ 1200 4910
 $Comp
-L Device:Polyfuse F1
+L Bast-Pro-Mini-M0-rescue:Polyfuse-Device F1
 U 1 1 5BB4BE5F
 P 1910 4200
@@
 	2260 4200 2260 4070
 $Comp
-L Device:C_Small C1
+L Bast-Pro-Mini-M0-rescue:C_Small-Device C1
 U 1 1 5BB50FD7
 P 8010 4850
@@
 $EndComp
 $Comp
-L Bast-Pro-Mini-M0-rescue:AP2112K-3.3TRG1-Croketa-cache U1
+L Bast-Pro-Mini-M0-rescue:AP2112K-3.3TRG1-Croketa-cache-Bast-Pro-Mini-M0-rescue U1
 U 1 1 5BB540C8
 P 9060 4720
@@
 $EndComp
 $Comp
-L Device:C_Small C2
+L Bast-Pro-Mini-M0-rescue:C_Small-Device C2
 U 1 1 5BB62453
 P 10150 4670
@@
 	9950 4520 10150 4520
 $Comp
-L Switch:SW_DPST_x2 SW1
+L Bast-Pro-Mini-M0-rescue:SW_DPST_x2-Switch SW1
 U 1 1 5BB741E9
 P 10145 1730
@@
 	3950 1410 4430 1410
 $Comp
-L Connector_Generic:Conn_02x02_Odd_Even J2
+L Bast-Pro-Mini-M0-rescue:Conn_02x02_Odd_Even-Connector_Generic J2
 U 1 1 5BB5EF14
 P 4315 4290
@@
 LED
 $Comp
-L Bast-Pro-Mini-M0-rescue:+3.3V-Croketa-cache #PWR0101
+L Bast-Pro-Mini-M0-rescue:+3.3V-Croketa-cache-Bast-Pro-Mini-M0-rescue #PWR0101
 U 1 1 5BBD0E40
 P 2630 1170
